File: trim.kicad_sch (KiCad schematic)
At the start: 0 parts

Commit message: Made trim circuit
Parts:
- added C37: 2.2uF, symbol Device:C
- added C38: 100nF, symbol Device:C
- added C39: 1uF, symbol Device:C
- added C40: 1nF, symbol Device:C
- added R22: 400ohm, symbol Device:R
- added R23: 51kOhm, symbol Device:R
- added R24: 50kOhm, symbol Device:R
- added U4: MAX4238AUT, Package_TO_SOT_SMD:SOT-23-6, symbol Amplifier_Operational:MAX4238AUT
- added U7: TCLT1003, SOP-4L_TC, symbol 2026-03-24_13-08-40:TCLT1003
- added U8: ADR361AUJZ-REEL7, UJ_5_ADI, symbol 2026-03-24_13-55-25:ADR361AUJZ-REEL7
Connections:
- new net: C38.1, U4.3 (+), U8.4 (VOUT)
- new net: C37.2, R22.1, U4.1
- new net: R22.2, U7.2 (C)
- new net: C37.1, R23.2, U4.4 (-)
- new net +5V: C39.1, U4.5 (~{SHDN}), U4.6 (V+), U7.1 (A), U8.3 (VIN)
- new net GNDA: C38.2, C39.2, U4.2 (V-), U8.2 (GND)
- new net GNDD: C40.2, R24.2, U7.3 (E)
- new net TR1: C40.1, R24.1, U7.4 (C)
- new net VoltageSense: R23.1
- no-connect marks 0 -> 1
Other:
- note added: "1uF-10uF"
- note added: "2.5V reference"
- note added: "optocoupler"

Commit message: assigned footprints, some minor schematic stuff, started layout
Parts:
- added R603, R604: 301ohm, Resistor_SMD:R_0603_1608Metric, symbol Device:R
- C601: renamed from C38; footprint (none) -> Capacitor_SMD:C_0603_1608Metric
- C602: renamed from C39; footprint (none) -> Capacitor_SMD:C_0603_1608Metric
- C603: renamed from C37; footprint (none) -> Capacitor_SMD:C_0603_1608Metric
- C604: renamed from C40; footprint (none) -> Capacitor_SMD:C_0603_1608Metric
- R601: renamed from R23; footprint (none) -> Resistor_SMD:R_0603_1608Metric
- R602: renamed from R22; footprint (none) -> Resistor_SMD:R_0603_1608Metric
- R605: renamed from R24; footprint (none) -> Resistor_SMD:R_0603_1608Metric
- U601: renamed from U8; footprint UJ_5_ADI -> footprints:UJ_5_ADI
- U603: renamed from U7; footprint SOP-4L_TC -> footprints:SOP-4L_TC
- renumbered U4 to U602
Connections:
- net TR1: now also R603.1; no longer C604.1, R605.1, U603.4 (C)
- net GNDD renamed GNDPWR
- new net: C604.1, R603.2, R604.2, R605.1, U603.4 (C)
- new net TR2: R604.1
