File: uC.kicad_sch (KiCad schematic)
At the start: 23 parts, among them J201 5023860270, J202 Conn_01x05, J203 Conn_01x04, J204 Conn_01x04, U201 STM32G431KBT6, Y201 ECS-2520MV-xxx-xx

Commit message: Layout done except for silkscreen
Parts:
- removed NT1: NetTie_2, NetTie:NetTie-2_SMD_Pad2.0mm, symbol Device:NetTie_2
- renumbered C208 to C207, C207 to C208
Changed lines of the file:
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@@
 	)
 	(junction
-		(at 158.115 137.16)
-		(diameter 0)
-		(color 0 0 0 0)
-	)
-	(junction
 		(at 246.38 55.88)
 		(diameter 0)
@@
 	(wire
 		(pts
+			(xy 161.29 137.16) (xy 161.29 144.78)
+		)
+		(stroke
+			(width 0)
+			(type default)
+		)
+	)
+	(wire
+		(pts
 			(xy 58.42 106.68) (xy 58.42 113.03)
 		)
@@
 	(wire
 		(pts
-			(xy 156.21 142.24) (xy 158.115 142.24)
-		)
-		(stroke
-			(width 0)
-			(type default)
-		)
-	)
-	(wire
-		(pts
 			(xy 156.21 83.82) (xy 162.56 83.82)
 		)
@@
 	(wire
 		(pts
-			(xy 163.83 114.3) (xy 163.83 111.76)
+			(xy 156.21 137.16) (xy 161.29 137.16)
 		)
 		(stroke
@@
 	(wire
 		(pts
-			(xy 156.21 142.24) (xy 156.21 144.78)
+			(xy 163.83 114.3) (xy 163.83 111.76)
 		)
 		(stroke
@@
 	(wire
 		(pts
-			(xy 158.115 137.16) (xy 165.1 137.16)
+			(xy 156.21 142.24) (xy 156.21 144.78)
 		)
 		(stroke
@@
 	(wire
 		(pts
-			(xy 156.21 137.16) (xy 158.115 137.16)
-		)
-		(stroke
-			(width 0)
-			(type default)
-		)
-	)
-	(wire
-		(pts
 			(xy 172.72 63.5) (xy 198.12 63.5)
 		)
@@
 		(in_pos_files yes)
 		(dnp no)
-		(property "Reference" "C207"
+		(property "Reference" "C208"
 			(at 245.11 100.33 0)
 			(show_name no)
@@
 			(project "LV_DCDC"
 				(path "/ccad4640-78c7-423b-83df-3ec0b90aa2b3/f9342e9a-2c81-4a9f-bedf-76ac3e437a63"
-					(reference "C207")
+					(reference "C208")
 					(unit 1)
 				)
@@
 		(dnp no)
 		(fields_autoplaced yes)
-		(property "Reference" "#PWR0227"
+		(property "Reference" "#PWR0216"
 			(at 185.42 64.77 0)
 			(hide yes)
@@
 			(project "LV_DCDC"
 				(path "/ccad4640-78c7-423b-83df-3ec0b90aa2b3/f9342e9a-2c81-4a9f-bedf-76ac3e437a63"
-					(reference "#PWR0227")
+					(reference "#PWR0216")
 					(unit 1)
 				)
@@
 		(dnp no)
 		(fields_autoplaced yes)
-		(property "Reference" "#PWR0223"
+		(property "Reference" "#PWR0225"
 			(at 260.35 69.85 0)
 			(hide yes)
@@
 			(project "LV_DCDC"
 				(path "/ccad4640-78c7-423b-83df-3ec0b90aa2b3/f9342e9a-2c81-4a9f-bedf-76ac3e437a63"
-					(reference "#PWR0223")
+					(reference "#PWR0225")
 					(unit 1)
 				)
@@
 		(dnp no)
 		(fields_autoplaced yes)
-		(property "Reference" "#PWR0224"
+		(property "Reference" "#PWR0226"
 			(at 266.7 52.07 0)
 			(hide yes)
@@
 			(project "LV_DCDC"
 				(path "/ccad4640-78c7-423b-83df-3ec0b90aa2b3/f9342e9a-2c81-4a9f-bedf-76ac3e437a63"
-					(reference "#PWR0224")
+					(reference "#PWR0226")
 					(unit 1)
 				)
@@
 		(dnp no)
 		(fields_autoplaced yes)
-		(property "Reference" "C208"
+		(property "Reference" "C207"
 			(at 201.93 71.1199 0)
 			(show_name no)
@@
 			(project "LV_DCDC"
 				(path "/ccad4640-78c7-423b-83df-3ec0b90aa2b3/f9342e9a-2c81-4a9f-bedf-76ac3e437a63"
-					(reference "C208")
+					(reference "C207")
 					(unit 1)
 				)
@@
 		(dnp no)
 		(fields_autoplaced yes)
-		(property "Reference" "#PWR0216"
+		(property "Reference" "#PWR0218"
 			(at 198.12 64.77 0)
 			(hide yes)
@@
 			(project "LV_DCDC"
 				(path "/ccad4640-78c7-423b-83df-3ec0b90aa2b3/f9342e9a-2c81-4a9f-bedf-76ac3e437a63"
-					(reference "#PWR0216")
+					(reference "#PWR0218")
 					(unit 1)
 				)
@@
 		(dnp no)
 		(fields_autoplaced yes)
-		(property "Reference" "#PWR0225"
+		(property "Reference" "#PWR0227"
 			(at 266.7 111.76 0)
 			(hide yes)
@@
 			(project "LV_DCDC"
 				(path "/ccad4640-78c7-423b-83df-3ec0b90aa2b3/f9342e9a-2c81-4a9f-bedf-76ac3e437a63"
-					(reference "#PWR0225")
+					(reference "#PWR0227")
 					(unit 1)
 				)
@@
 		(in_pos_files yes)
 		(dnp no)
-		(property "Reference" "#PWR0218"
+		(property "Reference" "#PWR0220"
 			(at 205.74 85.09 0)
 			(hide yes)
@@
 			(project "LV_DCDC"
 				(path "/ccad4640-78c7-423b-83df-3ec0b90aa2b3/f9342e9a-2c81-4a9f-bedf-76ac3e437a63"
-					(reference "#PWR0218")
+					(reference "#PWR0220")
 					(unit 1)
 				)
@@
 		(in_pos_files yes)
 		(dnp no)
-		(property "Reference" "#PWR0222"
+		(property "Reference" "#PWR0224"
 			(at 259.08 44.45 0)
 			(hide yes)
@@
 			(project "LV_DCDC"
 				(path "/ccad4640-78c7-423b-83df-3ec0b90aa2b3/f9342e9a-2c81-4a9f-bedf-76ac3e437a63"
-					(reference "#PWR0222")
+					(reference "#PWR0224")
 					(unit 1)
 				)
@@
 	)
 	(symbol
-		(lib_id "Device:NetTie_2")
-		(at 158.115 139.7 90)
-		(unit 1)
-		(body_style 1)
-		(exclude_from_sim no)
-		(in_bom no)
-		(on_board yes)
-		(in_pos_files yes)
-		(dnp no)
-		(fields_autoplaced yes)
-		(property "Reference" "NT1"
-			(at 160.02 138.4299 90)
-			(show_name no)
-			(do_not_autoplace no)
-			(effects
-				(font
-					(size 1.27 1.27)
-				)
-				(justify right)
-			)
-		)
-		(property "Value" "NetTie_2"
-			(at 160.02 140.9699 90)
-			(show_name no)
-			(do_not_autoplace no)
-			(effects
-				(font
-					(size 1.27 1.27)
-				)
-				(justify right)
-			)
-		)
-		(property "Footprint" "NetTie:NetTie-2_SMD_Pad2.0mm"
-			(at 158.115 139.7 0)
-			(hide yes)
-			(show_name no)
-			(do_not_autoplace no)
-			(effects
-				(font
-					(size 1.27 1.27)
-				)
-			)
-		)
-		(property "Datasheet" ""
-			(at 158.115 139.7 0)
-			(hide yes)
-			(show_name no)
-			(do_not_autoplace no)
-			(effects
-				(font
-					(size 1.27 1.27)
-				)
-			)
-		)
-		(property "Description" "Net tie, 2 pins"
-			(at 158.115 139.7 0)
-			(hide yes)
-			(show_name no)
-			(do_not_autoplace no)
-			(effects
-				(font
-					(size 1.27 1.27)
-				)
-			)
-		)
-		(pin "2"
-		)
-		(pin "1"
-		)
-		(instances
-			(project "LV_DCDC"
-				(path "/ccad4640-78c7-423b-83df-3ec0b90aa2b3/f9342e9a-2c81-4a9f-bedf-76ac3e437a63"
-					(reference "NT1")
-					(unit 1)
-				)
-			)
-		)
-	)
-	(symbol
 		(lib_id "Connector_Generic:Conn_01x04")
 		(at 278.13 100.33 0)
@@
 		(dnp no)
 		(fields_autoplaced yes)
-		(property "Reference" "#PWR0220"
+		(property "Reference" "#PWR0222"
 			(at 251.46 96.52 0)
 			(hide yes)
@@
 			(project "LV_DCDC"
 				(path "/ccad4640-78c7-423b-83df-3ec0b90aa2b3/f9342e9a-2c81-4a9f-bedf-76ac3e437a63"
-					(reference "#PWR0220")
+					(reference "#PWR0222")
 					(unit 1)
 				)
@@
 		(dnp no)
 		(fields_autoplaced yes)
-		(property "Reference" "#PWR0211"
+		(property "Reference" "#PWR0212"
 			(at 162.56 97.79 0)
 			(hide yes)
@@
 			(project "LV_DCDC"
 				(path "/ccad4640-78c7-423b-83df-3ec0b90aa2b3/f9342e9a-2c81-4a9f-bedf-76ac3e437a63"
-					(reference "#PWR0211")
+					(reference "#PWR0212")
 					(unit 1)
 				)
@@
 		(in_pos_files yes)
 		(dnp no)
-		(property "Reference" "#PWR0219"
+		(property "Reference" "#PWR0221"
 			(at 246.38 44.45 0)
 			(hide yes)
@@
 			(project "LV_DCDC"
 				(path "/ccad4640-78c7-423b-83df-3ec0b90aa2b3/f9342e9a-2c81-4a9f-bedf-76ac3e437a63"
-					(reference "#PWR0219")
+					(reference "#PWR0221")
 					(unit 1)
 				)
@@
 	(symbol
 		(lib_id "power:GNDA")
-		(at 165.1 137.16 0)
+		(at 161.29 144.78 0)
 		(unit 1)
 		(body_style 1)
@@
 		(in_pos_files yes)
 		(dnp no)
-		(property "Reference" "#PWR0212"
-			(at 165.1 143.51 0)
+		(property "Reference" "#PWR0211"
+			(at 161.29 151.13 0)
 			(hide yes)
 			(show_name no)
@@
 		)
 		(property "Value" "GNDA"
-			(at 165.1 140.97 0)
+			(at 161.29 148.59 0)
 			(show_name no)
 			(do_not_autoplace no)
@@
 		)
 		(property "Footprint" ""
-			(at 165.1 137.16 0)
+			(at 161.29 144.78 0)
 			(hide yes)
 			(show_name no)
@@
 		)
 		(property "Datasheet" ""
-			(at 165.1 137.16 0)
+			(at 161.29 144.78 0)
 			(hide yes)
 			(show_name no)
@@
 		)
 		(property "Description" "Power symbol creates a global label with name \"GNDA\" , analog ground"
-			(at 165.1 137.16 0)
+			(at 161.29 144.78 0)
 			(hide yes)
 			(show_name no)
@@
 			(project "LV_DCDC"
 				(path "/ccad4640-78c7-423b-83df-3ec0b90aa2b3/f9342e9a-2c81-4a9f-bedf-76ac3e437a63"
-					(reference "#PWR0212")
+					(reference "#PWR0211")
 					(unit 1)
 				)
@@
 		(dnp no)
 		(fields_autoplaced yes)
-		(property "Reference" "#PWR0221"
+		(property "Reference" "#PWR0223"
 			(at 251.46 111.76 0)
 			(hide yes)
@@
 			(project "LV_DCDC"
 				(path "/ccad4640-78c7-423b-83df-3ec0b90aa2b3/f9342e9a-2c81-4a9f-bedf-76ac3e437a63"
-					(reference "#PWR0221")
+					(reference "#PWR0223")
 					(unit 1)
 				)
@@
 		(dnp no)
 		(fields_autoplaced yes)
-		(property "Reference" "#PWR0226"
+		(property "Reference" "#PWR0219"
 			(at 198.12 82.55 0)
 			(hide yes)
@@
 			(project "LV_DCDC"
 				(path "/ccad4640-78c7-423b-83df-3ec0b90aa2b3/f9342e9a-2c81-4a9f-bedf-76ac3e437a63"
-					(reference "#PWR0226")
+					(reference "#PWR0219")
 					(unit 1)
 				)
